File: kicad_proj/eval-board-1_buck-regulator/eval-board-1_buck-regulator.kicad_sch (KiCad schematic)
At the start: 1 part

Commit message: Updates from the first stream
Parts:
- added C1, C2: GCJ32EC71E226KE02, footprints:CAPACITOR_1210N, symbol eval-board-1_buck-regulator:GCJ32EC71E226KE02
- added C10, C11, C7, C8, C9: 10u, symbol Device:C
- added C3: 100uF, symbol Device:CP
- added C4: 4.7u, symbol Device:C
- added C5: 1u, symbol Device:C
- added C6: 0.1uF, symbol Device:C
- added D1, D2: LED, symbol Device:LED
- added FB1: Ferrite_Bead, symbol Device:Ferrite_Bead
- added J1, J3: Conn_01x02, symbol Connector_Generic:Conn_01x02
- added J2: Conn_01x06, symbol Connector_Generic:Conn_01x06
- added JP1: Jumper_NC_Dual, symbol Device:Jumper_NC_Dual
- added JP2: Jumper, symbol Device:Jumper
- added L1: 1uH, symbol Device:L
- added R1, R2, R4, R7: 10K, symbol Device:R_US
- added R10: 220, symbol Device:R_US
- added R3: 510, symbol Device:R_US
- added R5, R6, R8: 8.87K, symbol Device:R_US
- added R9: 2.2, symbol Device:R_US
- added TP1, TP2: TestPoint, symbol Connector:TestPoint
- gave numbers to parts that had none: 1
Connections:
- net at U1.1 (PVIN): now also U1.2 (PVIN), U1.23 (VIN), U1.3 (PVIN), U1.34 (PVIN), C2.1, C3.1, FB1.2
- net GND: now reaches U1.11 (VSEN-)
- net GND: now also U1.16 (AGND), U1.32 (PGND), U1.33 (PGND), U1.7 (AGND), C1.2, C10.2, C11.2, C2.2, C3.2, C4.2, C5.2, C7.2, C8.2, C9.2, D1.1 (K), D2.1 (K), J1.1 (Pin_1), J2.1 (Pin_1), J3.1 (Pin_1), JP2.1, R5.2, R6.2, R8.2
- net +5V: now reaches U1.12 (VSEN+)
- net +5V: now also C10.1, C11.1, C7.1, C8.1, C9.1, J3.2 (Pin_2), L1.2, R10.1
- net PGOOD: now reaches U1.13 (PGOOD)
- net PGOOD: now also J2.2 (Pin_2), R7.2
- net at U1.14 (ADDR): now also R5.1
- net at U1.15 (VSET): now also R8.1
- net at U1.17 (RT/SYNC): now also R6.1
- net SALERT: now reaches U1.18 (SALRT)
- net SALERT: now also J2.6 (Pin_6)
- net SDA: now reaches U1.19 (SDA)
- net SDA: now also J2.4 (Pin_4), R2.2
- net SCL: now reaches U1.20 (SCL)
- net SCL: now also J2.5 (Pin_5), R1.2
- net EN: now reaches U1.21 (EN)
- net EN: now also JP2.2, R4.2
- net VDD: now reaches U1.22 (VDD)
- net VDD: now also C5.1, JP1.1, R4.1
- net at U1.24 (PVCC): now also C4.1
- net at U1.25 (GL): now also TP2.1
- net at U1.26 (SW): now also U1.27 (SW), U1.28 (SW), U1.29 (SW), U1.30 (SW), U1.31 (SW), L1.1
- net at U1.4 (PH): now also R9.2
- net at U1.5 (GH): now also TP1.1
- net at U1.6 (BOOT): now also C6.1
- new net: C6.2, R9.1
- new net: D1.2 (A), R3.2
- new net: D2.2 (A), R10.2
- new net +12V: C1.1, FB1.1, J1.2 (Pin_2), R3.1
- new net EXTERN_VTG: J2.3 (Pin_3), JP1.3
- new net PULLUP_VTG: JP1.2, R1.1, R2.1, R7.1
Other:
- note added: "EXTERNAL (3v3) DISABLES PULLUPS IF NO VTG SUPPLIED"
- note added: "FREQ = 1MHz OUTPUT VTG = 5V ADDR = C"
- note added: "ONBOARD 5V"
- note added: "i2c PULLUPS"
- moved on the sheet: U1

Commit message: Updates from livestream
Parts:
- removed C1, C2: GCJ32EC71E226KE02, footprints:CAPACITOR_1210N, symbol eval-board-1_buck-regulator:GCJ32EC71E226KE02
- removed C10: 10u, symbol Device:C
- added C1, C17, C18, C4: GRM32ER71C226KEA8, eval-board-1_buck-regulator:CAPACITOR_1210N, symbol Device:C
- added C13, C5, C6: GRM32ER71E226ME15K, eval-board-1_buck-regulator:CAPACITOR_1210N, symbol Device:C
- added C14: GRM188R61H225ME11D, eval-board-1_buck-regulator:CAPACITOR_0603N, symbol Device:C
- added C3: UCH1V470MCS1GS, eval-board-1_buck-regulator:CAPAE660X580L260X65N, symbol Device:CP
- added C7: GRM188R61H225ME11D, footprints:CAPACITOR_0603N, symbol capacitors:GRM188R61H225ME11D
- added R1, R2, R4: 220, eval-board-1_buck-regulator:CAPACITOR_0402N, symbol Device:R_US
- added R12, R13: 10K, eval-board-1_buck-regulator:CAPACITOR_0402N, symbol Device:R_US
- C10: renamed from C4; footprint (none) -> eval-board-1_buck-regulator:CAPACITOR_0603N
- C11, C8, C9: value 10u -> GRM32ER71E226ME15K; footprint (none) -> eval-board-1_buck-regulator:CAPACITOR_1210N; id (none) -> 22uF
- C12: renamed from C5; footprint (none) -> eval-board-1_buck-regulator:CAPACITOR_0402N
- C15: renamed from C6; footprint (none) -> eval-board-1_buck-regulator:CAPACITOR_0402N
- C16: renamed from C7; value 10u -> GRM32ER71C226KEA8; footprint (none) -> eval-board-1_buck-regulator:CAPACITOR_1210N; id (none) -> 22uF
- C2: renamed from C3; value 100uF -> UCH1V470MCS1GS; footprint (none) -> eval-board-1_buck-regulator:CAPAE660X580L260X65N; id (none) -> 47uF
- D1, D2: footprint (none) -> eval-board-1_buck-regulator:CAPACITOR_0603N
- FB1: value Ferrite_Bead -> 74279221100; footprint (none) -> eval-board-1_buck-regulator:CAPACITOR_1206N
- J1, J3, JP2: footprint (none) -> Connector_PinHeader_2.54mm:PinHeader_1x02_P2.54mm_Vertical
- J2: footprint (none) -> Connector_PinHeader_2.54mm:PinHeader_1x06_P2.54mm_Vertical
- JP1: footprint (none) -> Connector_PinHeader_2.54mm:PinHeader_1x03_P2.54mm_Vertical
- L1: value 1uH -> PA4343.102NLT; footprint (none) -> eval-board-1_buck-regulator:PA4343_PM4343; id (none) -> 1uH
- R10: renamed from R7; footprint (none) -> eval-board-1_buck-regulator:CAPACITOR_0402N
- R11: renamed from R8; footprint (none) -> eval-board-1_buck-regulator:CAPACITOR_0402N
- R14: renamed from R9; footprint (none) -> eval-board-1_buck-regulator:CAPACITOR_0402N
- R15: renamed from R10; footprint (none) -> eval-board-1_buck-regulator:CAPACITOR_0402N
- R3: renamed from R1; footprint (none) -> eval-board-1_buck-regulator:CAPACITOR_0402N
- R5: renamed from R2; footprint (none) -> eval-board-1_buck-regulator:CAPACITOR_0402N
- R6: renamed from R3; footprint (none) -> eval-board-1_buck-regulator:CAPACITOR_0402N
- R7: renamed from R4; footprint (none) -> eval-board-1_buck-regulator:CAPACITOR_0402N
- R8: renamed from R5; footprint (none) -> eval-board-1_buck-regulator:CAPACITOR_0402N
- R9: renamed from R6; footprint (none) -> eval-board-1_buck-regulator:CAPACITOR_0402N
- TP1, TP2: footprint (none) -> TestPoint:TestPoint_Pad_1.5x1.5mm
Connections:
- net +12V: now also C1.1
- net +5V: now also C17.1, C18.1, R12.2; no longer C11.1, C8.1, C9.1, U1.12 (VSEN+)
- net GND: now also C1.2, C13.2, C14.2, C17.2, C18.2, C3.2, C4.2, C5.2, C6.2, C7.2, R13.2; no longer U1.11 (VSEN-)
- net SALERT: now also R1.2; no longer J2.6 (Pin_6)
- net SCL: now also R4.2; no longer J2.5 (Pin_5)
- net SDA: now also R2.2; no longer J2.4 (Pin_4)
- net at C2.1, FB1.2, U1.1 (PVIN)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: now also C11.1, C8.1, C9.1, C13.1, C14.1, C3.1, C4.1, C5.1, C6.1, C7.1
- new net: J2.6 (Pin_6), R1.1
- new net: J2.4 (Pin_4), R2.1
- new net: J2.5 (Pin_5), R4.1
- new net: R13.1, U1.11 (VSEN-)
- new net: R12.1, U1.12 (VSEN+)
Other:
- moved on the sheet: C2, FB1, R7

Commit message: Livestream updates
Parts:
- removed C4: GRM32ER71C226KEA8, eval-board-1_buck-regulator:CAPACITOR_1210N, symbol Device:C
- added C19, C4: UCH1V470MCS1GS, eval-board-1_buck-regulator:CAPAE660X580L260X65N, symbol Device:CP
- added H1, H2, H3: MountingHole_Pad, MountingHole:MountingHole_2.7mm_M2.5_Pad_Via, symbol Mechanical:MountingHole_Pad
- J1, J3: footprint Connector_PinHeader_2.54mm:PinHeader_1x02_P2.54mm_Vertical -> eval-board-1_buck-regulator:1935776
- renumbered R2 to R1, R3 to R2, R1 to R3
Connections:
- net +5V: now also C19.1
- net EXTERN_VTG: now also J2.6 (Pin_6); no longer J2.3 (Pin_3)
- net GND: now also C19.2, C4.2, H1.1, H2.1, H3.1
- net at C11.1, C13.1, C14.1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: now also C4.1
- net at R3.1: now also J2.3 (Pin_3); no longer J2.6 (Pin_6)
Other:
- moved on the sheet: R3
